Commit message: cleaned up urdf.xacro model
- added consistent labels
- moved stuff around

File: mayday_control/scripts/test_mayday_robot_data/DescriptionTestCase/mayday.urdf.xacro (robot description, xacro)
@@ -30,4 +30,5 @@
   <xacro:property name="tibia_z" value="0.01" />
   <xacro:property name="tibia_weight" value="0.05" />
+  <!-- materials -->
   <material name="black">
     <color rgba="0 0 0 1"/>
@@ -68,4 +69,225 @@
     </link>
   </xacro:macro>
+  <!-- coxa macro  -->
+  <xacro:macro name="coxa" params="prefix">
+    <link name="${prefix}_coxa">
+      <visual>
+        <geometry>
+          <box size="${coxa_x} ${coxa_y} ${coxa_z}"/>
+        </geometry>
+        <origin xyz="${(coxa_x/2-dynamixel_y/2)} 0 0" rpy="0 0 0"/>
+        <material name="grey"/>
+      </visual>
+      <collision>
+        <geometry>
+          <box size="${coxa_x} ${coxa_y} ${coxa_z}"/>
+        </geometry>
+        <origin xyz="${coxa_x/2-dynamixel_y/2} 0 0" rpy="0 0 0"/>
+      </collision>
+      <xacro:box_inertial mass="${coxa_weight}" x="${coxa_x}" y="${coxa_y}" z="${coxa_z}"
+                          x_="${coxa_x/2-dynamixel_y/2}" y_="0" z_="0"/>
+    </link>
+  </xacro:macro>
+  <!-- femur macro  -->
+  <xacro:macro name="femur" params="prefix">
+    <link name="${prefix}_femur">
+      <visual>
+        <geometry>
+          <box size="${femur_x} ${femur_y} ${femur_z}"/>
+        </geometry>
+        <origin xyz="${femur_x/2-dynamixel_y/2} 0 0" rpy="0 0 0"/>
+        <material name="grey"/>
+      </visual>
+      <collision>
+        <geometry>
+          <box size="${femur_x} ${femur_y} ${femur_z}"/>
+        </geometry>
+        <origin xyz="${femur_x/2-dynamixel_y/2} 0 0" rpy="0 0 0"/>
+      </collision>
+      <xacro:box_inertial mass="${femur_weight}" x="${femur_x}" y="${femur_y}" z="${femur_z}"
+                          x_="${femur_x/2-dynamixel_y/2}" y_="0" z_="0"/>
+    </link>
+  </xacro:macro>
+  <!-- leg macro  -->
+  <xacro:macro name="leg" params="prefix x_offset yaw_offset reflect">
+    <!-- coxa_dynamixel  -->
+    <xacro:dynamixel prefix="${prefix}_coxa" />
+    <joint name="${prefix}_thorax_to_coxa_dynamixel_joint" type="fixed">
+      <parent link="thorax"/>
+      <child link="${prefix}_coxa_dynamixel"/>
+      <origin xyz="${x_offset} ${reflect*thorax_y/2} 0" rpy="0 0 ${reflect*yaw_offset}"/>
+    </joint>
+    <!-- top_coxa -->
+    <xacro:coxa prefix="${prefix}_top" />
+    <joint name="${prefix}_coxa_dynamixel_to_top_coxa_joint" type="revolute">
+      <axis xyz="0 0 1"/>
+      <limit effort="1.5" lower="${-tau*1/8}" upper="${tau*1/8}" velocity="${2*tau}"/>
+      <parent link="${prefix}_coxa_dynamixel"/>
+      <child link="${prefix}_top_coxa"/>
+      <origin xyz="0 0 ${dynamixel_z/2 + coxa_z/2 + tolerance}" rpy="0 0 0" />
+      <dynamics damping="0.01" friction="0.1"/>
+    </joint>
+    <transmission name="${prefix}_coxa_dynamixel_to_top_coxa_joint_transmission">
+      <type>transmission_interface/SimpleTransmission</type>
+      <joint name="${prefix}_coxa_dynamixel_to_top_coxa_joint">
+        <hardwareInterface>hardware_interface/EffortJointInterface</hardwareInterface>
+      </joint>
+      <actuator name="${prefix}_coxa_dynamixel_to_top_coxa_joint_motor">
+        <hardwareInterface>hardware_interface/EffortJointInterface</hardwareInterface>
+        <mechanicalReduction>1</mechanicalReduction>
+      </actuator>
+    </transmission>
+    <!-- bottom_coxa  -->
+    <xacro:coxa prefix="${prefix}_bottom" />
+    <joint name="${prefix}_femur_dynamixel_to_bottom_coxa_joint" type="fixed">
+      <parent link="${prefix}_top_coxa"/>
+      <child link="${prefix}_bottom_coxa"/>
+      <origin xyz="0 0 ${-(dynamixel_z+coxa_z+tolerance*2)}" rpy="${tau/2} 0 0"/>
+    </joint>
+    <!-- femur_dynamixel  -->
+    <xacro:dynamixel prefix="${prefix}_femur" />
+    <joint name="${prefix}_top_coxa_to_femur_dynamixel_joint" type="fixed">
+      <parent link="${prefix}_top_coxa"/>
+      <child link="${prefix}_femur_dynamixel"/>
+      <origin xyz="${coxa_x/2 - dynamixel_y/2  +  coxa_x/2 - dynamixel_y/2 + tolerance/2} 0 ${-(dynamixel_x/2 + coxa_z/2)}" rpy="${-tau/4} ${tau/4} 0"/>
+    </joint>
+    <!-- left_femur -->
+    <xacro:femur prefix="${prefix}_left" />
+    <joint name="${prefix}_femur_dynamixel_to_left_femur_joint" type="revolute">
+      <axis xyz="0 0 1"/>
+      <limit effort="1.5" lower="${-tau*3/8}" upper="${tau*3/8}" velocity="${2*tau}"/>
+      <parent link="${prefix}_femur_dynamixel"/>
+      <child link="${prefix}_left_femur"/>
+      <origin xyz="0 0 ${dynamixel_z/2 + femur_z/2 + tolerance}" rpy="0 0 ${-tau/4}" />
+      <dynamics damping="0.01" friction="0.1"/>
+    </joint>
+    <transmission name="${prefix}_femur_dynamixel_to_left_femur_joint_transmission">
+      <type>transmission_interface/SimpleTransmission</type>
+      <joint name="${prefix}_femur_dynamixel_to_left_femur_joint">
+        <hardwareInterface>hardware_interface/EffortJointInterface</hardwareInterface>
+      </joint>
+      <actuator name="${prefix}_femur_dynamixel_to_left_femur_joint_motor">
+        <hardwareInterface>hardware_interface/EffortJointInterface</hardwareInterface>
+        <mechanicalReduction>1</mechanicalReduction>
+      </actuator>
+    </transmission>
+    <!-- right_femur  -->
+    <xacro:femur prefix="${prefix}_right" />
+    <joint name="${prefix}_left_femur_to_right_femur_joint" type="fixed">
+      <parent link="${prefix}_left_femur"/>
+      <child link="${prefix}_right_femur"/>
+      <origin xyz="0 0 ${-(dynamixel_z + femur_z + tolerance*2)}" rpy="${tau/2} 0 0"/>
+    </joint>
+    <!-- tibia_dynamixel  -->
+    <xacro:dynamixel prefix="${prefix}_tibia" />
+    <joint name="${prefix}_left_femur_to_tibia_dynamixel_joint" type="revolute">
+      <parent link="${prefix}_left_femur"/>
+      <child link="${prefix}_tibia_dynamixel"/>
+      <origin xyz="${femur_x - dynamixel_y} 0 ${-(dynamixel_z/2 + femur_z/2 + tolerance)}" rpy="${tau/2} ${tau/2} 0" />
+      <axis xyz="0 0 1"/>
+      <limit effort="1.5" lower="${-tau*3/8}" upper="${tau*3/8}" velocity="${2*tau}"/>
+      <dynamics damping="0.01" friction="0.1"/>
+    </joint>
+    <transmission name="${prefix}_left_femur_to_tibia_dynamixel_joint_transmission">
+      <type>transmission_interface/SimpleTransmission</type>
+      <joint name="${prefix}_left_femur_to_tibia_dynamixel_joint">
+        <hardwareInterface>hardware_interface/EffortJointInterface</hardwareInterface>
+      </joint>
+      <actuator name="${prefix}_left_femur_to_tibia_dynamixel_joint_motor">
+        <hardwareInterface>hardware_interface/EffortJointInterface</hardwareInterface>
+        <mechanicalReduction>1</mechanicalReduction>
+      </actuator>
+    </transmission>
+    <!-- tibia -->
+    <link name="${prefix}_tibia">
+      <visual>
+        <geometry>
+          <box size="${tibia_x} ${tibia_y} ${tibia_z}"/>
+        </geometry>
+        <origin xyz="${tibia_x/2 - dynamixel_y/2 + dynamixel_z/2} 0 0" rpy="0 0 0"/>
+        <material name="grey"/>
+      </visual>
+      <collision>
+        <geometry>
+          <box size="${tibia_x} ${tibia_y} ${tibia_z}"/>
+        </geometry>
+        <origin xyz="${tibia_x/2 - dynamixel_y/2 + dynamixel_z/2} 0 0" rpy="0 0 0"/>
+      </collision>
+      <xacro:box_inertial mass="${tibia_weight}" x="${tibia_x}" y="${tibia_y}" z="${tibia_z}"
+                          x_="${tibia_x/2 - dynamixel_y/2 + dynamixel_z/2}" y_="0" z_="0"/>
+    </link>
+    <joint name="${prefix}_tibia_dynamixel_to_tibia_joint" type="fixed">
+      <parent link="${prefix}_tibia_dynamixel"/>
+      <child link="${prefix}_tibia"/>
+      <origin xyz="0 0 0" rpy="${tau/4} 0 ${tau/2}" />
+    </joint>
+    <!-- This block provides the simulator (Gazebo) with information on a few additional
+    physical properties. See http://gazebosim.org/tutorials/?tut=ros_urdf for more-->
+    <gazebo reference="${prefix}_top_coxa">
+      <mu1 value="0.2"/>
+      <mu2 value="0.2"/>
+      <kp value="10000000.0" />
+      <kd value="1.0" />
+      <material>Gazebo/Grey</material>
+      <selfCollide>True</selfCollide>
+    </gazebo>
+    <gazebo reference="${prefix}_bottom_coxa">
+      <mu1 value="0.2"/>
+      <mu2 value="0.2"/>
+      <kp value="10000000.0" />
+      <kd value="1.0" />
+      <material>Gazebo/Grey</material>
+      <selfCollide>True</selfCollide>
+    </gazebo>
+    <gazebo reference="${prefix}_right_femur">
+      <mu1 value="0.2"/>
+      <mu2 value="0.2"/>
+      <kp value="10000000.0" />
+      <kd value="1.0" />
+      <material>Gazebo/Grey</material>
+      <selfCollide>True</selfCollide>
+    </gazebo>
+    <gazebo reference="${prefix}_left_femur">
+      <mu1 value="0.2"/>
+      <mu2 value="0.2"/>
+      <kp value="10000000.0" />
+      <kd value="1.0" />
+      <material>Gazebo/Grey</material>
+      <selfCollide>True</selfCollide>
+    </gazebo>
+    <gazebo reference="${prefix}_tibia">
+      <mu1 value="0.2"/>
+      <mu2 value="0.2"/>
+      <kp value="10000000.0" />
+      <kd value="1.0" />
+      <material>Gazebo/Grey</material>
+      <selfCollide>True</selfCollide>
+    </gazebo>
+    <gazebo reference="${prefix}_coxa_dynamixel">
+      <mu1 value="0.2"/>
+      <mu2 value="0.2"/>
+      <kp value="10000000.0" />
+      <kd value="1.0" />
+      <material>Gazebo/Black</material>
+      <selfCollide>True</selfCollide>
+    </gazebo>
+    <gazebo reference="${prefix}_femur_dynamixel">
+      <mu1 value="0.2"/>
+      <mu2 value="0.2"/>
+      <kp value="10000000.0" />
+      <kd value="1.0" />
+      <material>Gazebo/Black</material>
+      <selfCollide>True</selfCollide>
+    </gazebo>
+    <gazebo reference="${prefix}_tibia_dynamixel">
+      <mu1 value="0.2"/>
+      <mu2 value="0.2"/>
+      <kp value="10000000.0" />
+      <kd value="1.0" />
+      <material>Gazebo/Black</material>
+      <selfCollide>True</selfCollide>
+    </gazebo>
+  </xacro:macro>
+  <!-- base_link  -->
   <link name="base_link">
   </link>
@@ -101,223 +323,4 @@
     <selfCollide>True</selfCollide>
   </gazebo>
-  <!-- coxa macro  -->
-  <xacro:macro name="coxa" params="prefix">
-    <link name="${prefix}_coxa">
-      <visual>
-        <geometry>
-          <box size="${coxa_x} ${coxa_y} ${coxa_z}"/>
-        </geometry>
-        <origin xyz="${(coxa_x/2-dynamixel_y/2)} 0 0" rpy="0 0 0"/>
-        <material name="grey"/>
-      </visual>
-      <collision>
-        <geometry>
-          <box size="${coxa_x} ${coxa_y} ${coxa_z}"/>
-        </geometry>
-        <origin xyz="${coxa_x/2-dynamixel_y/2} 0 0" rpy="0 0 0"/>
-      </collision>
-      <xacro:box_inertial mass="${coxa_weight}" x="${coxa_x}" y="${coxa_y}" z="${coxa_z}"
-                          x_="${coxa_x/2-dynamixel_y/2}" y_="0" z_="0"/>
-    </link>
-  </xacro:macro>
-  <!-- femur macro  -->
-  <xacro:macro name="femur" params="prefix">
-    <link name="${prefix}_femur">
-      <visual>
-        <geometry>
-          <box size="${femur_x} ${femur_y} ${femur_z}"/>
-        </geometry>
-        <origin xyz="${femur_x/2-dynamixel_y/2} 0 0" rpy="0 0 0"/>
-        <material name="grey"/>
-      </visual>
-      <collision>
-        <geometry>
-          <box size="${femur_x} ${femur_y} ${femur_z}"/>
-        </geometry>
-        <origin xyz="${femur_x/2-dynamixel_y/2} 0 0" rpy="0 0 0"/>
-      </collision>
-      <xacro:box_inertial mass="${femur_weight}" x="${femur_x}" y="${femur_y}" z="${femur_z}"
-                          x_="${femur_x/2-dynamixel_y/2}" y_="0" z_="0"/>
-    </link>
-  </xacro:macro>
-  <xacro:macro name="leg" params="prefix x_offset yaw_offset reflect">
-    <!-- coxa_dynamixel  -->
-    <xacro:dynamixel prefix="${prefix}_coxa" />
-    <joint name="${prefix}_thorax_to_coxa_dynamixel_joint" type="fixed">
-      <parent link="thorax"/>
-      <child link="${prefix}_coxa_dynamixel"/>
-      <origin xyz="${x_offset} ${reflect*thorax_y/2} 0" rpy="0 0 ${reflect*yaw_offset}"/>
-    </joint>
-    <!-- top_coxa -->
-    <xacro:coxa prefix="${prefix}_top" />
-    <joint name="${prefix}_coxa_dynamixel_to_top_coxa_joint" type="revolute">
-      <axis xyz="0 0 1"/>
-      <limit effort="1.5" lower="${-tau*1/8}" upper="${tau*1/8}" velocity="${2*tau}"/>
-      <parent link="${prefix}_coxa_dynamixel"/>
-      <child link="${prefix}_top_coxa"/>
-      <origin xyz="0 0 ${dynamixel_z/2 + coxa_z/2 + tolerance}" rpy="0 0 0" />
-      <dynamics damping="0.01" friction="0.1"/>
-    </joint>
-    <transmission name="${prefix}_coxa_dynamixel_to_top_coxa_joint_transmission">
-      <type>transmission_interface/SimpleTransmission</type>
-      <joint name="${prefix}_coxa_dynamixel_to_top_coxa_joint">
-        <hardwareInterface>hardware_interface/EffortJointInterface</hardwareInterface>
-      </joint>
-      <actuator name="${prefix}_coxa_dynamixel_to_top_coxa_joint_motor">
-        <hardwareInterface>hardware_interface/EffortJointInterface</hardwareInterface>
-        <mechanicalReduction>1</mechanicalReduction>
-      </actuator>
-    </transmission>
-    <!-- bottom_coxa  -->
-    <xacro:coxa prefix="${prefix}_bottom" />
-    <joint name="${prefix}_femur_dynamixel_to_bottom_coxa_joint" type="fixed">
-      <parent link="${prefix}_top_coxa"/>
-      <child link="${prefix}_bottom_coxa"/>
-      <origin xyz="0 0 ${-(dynamixel_z+coxa_z+tolerance*2)}" rpy="${tau/2} 0 0"/>
-    </joint>
-    <!-- femur_dynamixel  -->
-    <xacro:dynamixel prefix="${prefix}_femur" />
-    <joint name="${prefix}_top_coxa_to_femur_dynamixel_joint" type="fixed">
-      <parent link="${prefix}_top_coxa"/>
-      <child link="${prefix}_femur_dynamixel"/>
-      <origin xyz="${coxa_x/2 - dynamixel_y/2  +  coxa_x/2 - dynamixel_y/2 + tolerance/2} 0 ${-(dynamixel_x/2 + coxa_z/2)}" rpy="${-tau/4} ${tau/4} 0"/>
-    </joint>
-    <!-- left_femur -->
-    <xacro:femur prefix="${prefix}_left" />
-    <joint name="${prefix}_femur_dynamixel_to_left_femur_joint" type="revolute">
-      <axis xyz="0 0 1"/>
-      <limit effort="1.5" lower="${-tau*3/8}" upper="${tau*3/8}" velocity="${2*tau}"/>
-      <parent link="${prefix}_femur_dynamixel"/>
-      <child link="${prefix}_left_femur"/>
-      <origin xyz="0 0 ${dynamixel_z/2 + femur_z/2 + tolerance}" rpy="0 0 ${-tau/4}" />
-      <dynamics damping="0.01" friction="0.1"/>
-    </joint>
-    <transmission name="${prefix}_femur_dynamixel_to_left_femur_joint_transmission">
-      <type>transmission_interface/SimpleTransmission</type>
-      <joint name="${prefix}_femur_dynamixel_to_left_femur_joint">
-        <hardwareInterface>hardware_interface/EffortJointInterface</hardwareInterface>
-      </joint>
-      <actuator name="${prefix}_femur_dynamixel_to_left_femur_joint_motor">
-        <hardwareInterface>hardware_interface/EffortJointInterface</hardwareInterface>
-        <mechanicalReduction>1</mechanicalReduction>
-      </actuator>
-    </transmission>
-    <!-- right_femur  -->
-    <xacro:femur prefix="${prefix}_right" />
-    <joint name="${prefix}_left_femur_to_right_femur_joint" type="fixed">
-      <parent link="${prefix}_left_femur"/>
-      <child link="${prefix}_right_femur"/>
-      <origin xyz="0 0 ${-(dynamixel_z + femur_z + tolerance*2)}" rpy="${tau/2} 0 0"/>
-    </joint>
-    <!-- tibia_dynamixel  -->
-    <xacro:dynamixel prefix="${prefix}_tibia" />
-    <joint name="${prefix}_left_femur_to_tibia_dynamixel_joint" type="revolute">
-      <parent link="${prefix}_left_femur"/>
-      <child link="${prefix}_tibia_dynamixel"/>
-      <origin xyz="${femur_x - dynamixel_y} 0 ${-(dynamixel_z/2 + femur_z/2 + tolerance)}" rpy="${tau/2} ${tau/2} 0" />
-      <axis xyz="0 0 1"/>
-      <limit effort="1.5" lower="${-tau*3/8}" upper="${tau*3/8}" velocity="${2*tau}"/>
-      <dynamics damping="0.01" friction="0.1"/>
-    </joint>
-    <transmission name="${prefix}_left_femur_to_tibia_dynamixel_joint_transmission">
-      <type>transmission_interface/SimpleTransmission</type>
-      <joint name="${prefix}_left_femur_to_tibia_dynamixel_joint">
-        <hardwareInterface>hardware_interface/EffortJointInterface</hardwareInterface>
-      </joint>
-      <actuator name="${prefix}_left_femur_to_tibia_dynamixel_joint_motor">
-        <hardwareInterface>hardware_interface/EffortJointInterface</hardwareInterface>
-        <mechanicalReduction>1</mechanicalReduction>
-      </actuator>
-    </transmission>
-    <!-- tibia -->
-    <link name="${prefix}_tibia">
-      <visual>
-        <geometry>
-          <box size="${tibia_x} ${tibia_y} ${tibia_z}"/>
-        </geometry>
-        <origin xyz="${tibia_x/2 - dynamixel_y/2 + dynamixel_z/2} 0 0" rpy="0 0 0"/>
-        <material name="grey"/>
-      </visual>
-      <collision>
-        <geometry>
-          <box size="${tibia_x} ${tibia_y} ${tibia_z}"/>
-        </geometry>
-        <origin xyz="${tibia_x/2 - dynamixel_y/2 + dynamixel_z/2} 0 0" rpy="0 0 0"/>
-      </collision>
-      <xacro:box_inertial mass="${tibia_weight}" x="${tibia_x}" y="${tibia_y}" z="${tibia_z}"
-                          x_="${tibia_x/2 - dynamixel_y/2 + dynamixel_z/2}" y_="0" z_="0"/>
-    </link>
-    <joint name="${prefix}_tibia_dynamixel_to_tibia_joint" type="fixed">
-      <parent link="${prefix}_tibia_dynamixel"/>
-      <child link="${prefix}_tibia"/>
-      <origin xyz="0 0 0" rpy="${tau/4} 0 ${tau/2}" />
-    </joint>
-    <!-- This block provides the simulator (Gazebo) with information on a few additional
-    physical properties. See http://gazebosim.org/tutorials/?tut=ros_urdf for more-->
-    <gazebo reference="${prefix}_top_coxa">
-      <mu1 value="0.2"/>
-      <mu2 value="0.2"/>
-      <kp value="10000000.0" />
-      <kd value="1.0" />
-      <material>Gazebo/Grey</material>
-      <selfCollide>True</selfCollide>
-    </gazebo>
-    <gazebo reference="${prefix}_bottom_coxa">
-      <mu1 value="0.2"/>
-      <mu2 value="0.2"/>
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
Commit message: tau is built into xacro

File: mayday_control/scripts/test_mayday_robot_data/DescriptionTestCase/mayday.urdf.xacro (robot description, xacro)
@@ -8,5 +8,4 @@
   <xacro:property name="baselen" value="0.4" />
   <xacro:property name="wheeldiam" value="0.07" />
-  <xacro:property name="tau" value="${pi*2}" />
   <xacro:property name="tolerance" value="0.001" />
   <xacro:property name="dynamixel_x" value="0.0465" />
